Commit message: add urdf

File: resources/robots/go1/urdf/go1.urdf (robot description, URDF)
Before this commit: robot go1_description, 38 links, 37 joints
Links:
- removed link camera_chin
- removed link camera_face
- removed link camera_laserscan_link_left
- removed link camera_laserscan_link_right
- removed link camera_left
- removed link camera_optical_chin
- removed link camera_optical_face
- removed link camera_optical_left
- removed link camera_optical_rearDown
- removed link camera_optical_right
- removed link camera_rearDown
- removed link camera_right
- removed link ultraSound_face
- removed link ultraSound_left
- removed link ultraSound_right
- link FL_calf: mass 0.131 -> 0.158015; geometry collision box size=0.213 0.016 0.016; visual mesh filename=../meshes/calf.stl scale=1 1 1
- link FL_hip: mass 0.591 -> 0.510299; geometry collision cylinder length=0.04 radius=0.046; visual mesh filename=../meshes/hip.stl scale=1 1 1
- link FL_thigh: mass 0.92 -> 0.898919; geometry collision box size=0.213 0.0245 0.034; visual mesh filename=../meshes/thigh.stl scale=1 1 1
- link FL_thigh_shoulder: geometry 
- link FR_calf: mass 0.131 -> 0.158015; geometry collision box size=0.213 0.016 0.016; visual mesh filename=../meshes/calf.stl scale=1 1 1
- link FR_hip: mass 0.591 -> 0.510299; geometry collision cylinder length=0.04 radius=0.046; visual mesh filename=../meshes/hip.stl scale=1 1 1
- link FR_thigh: mass 0.92 -> 0.898919; geometry collision box size=0.213 0.0245 0.034; visual mesh filename=../meshes/thigh_mirror.stl scale=1 1 1
- link FR_thigh_shoulder: geometry 
- link RL_calf: mass 0.131 -> 0.158015; geometry collision box size=0.213 0.016 0.016; visual mesh filename=../meshes/calf.stl scale=1 1 1
- link RL_hip: mass 0.591 -> 0.510299; geometry collision cylinder length=0.04 radius=0.046; visual mesh filename=../meshes/hip.stl scale=1 1 1
- link RL_thigh: mass 0.92 -> 0.898919; geometry collision box size=0.213 0.0245 0.034; visual mesh filename=../meshes/thigh.stl scale=1 1 1
- link RL_thigh_shoulder: geometry 
- link RR_calf: mass 0.131 -> 0.158015; geometry collision box size=0.213 0.016 0.016; visual mesh filename=../meshes/calf.stl scale=1 1 1
- link RR_hip: mass 0.591 -> 0.510299; geometry collision cylinder length=0.04 radius=0.046; visual mesh filename=../meshes/hip.stl scale=1 1 1
- link RR_thigh: mass 0.92 -> 0.898919; geometry collision box size=0.213 0.0245 0.034; visual mesh filename=../meshes/thigh_mirror.stl scale=1 1 1
- link RR_thigh_shoulder: geometry 
- link imu_link: geometry visual box size=0.001 0.001 0.001
- link trunk: mass 5.204 -> 4.8; geometry collision box size=0.3762 0.0935 0.114; visual mesh filename=../meshes/trunk.stl scale=1 1 1
Joints:
- removed joint camera_joint_chin
- removed joint camera_joint_face
- removed joint camera_joint_left
- removed joint camera_joint_rearDown
- removed joint camera_joint_right
- removed joint camera_laserscan_joint_left
- removed joint camera_laserscan_joint_right
- removed joint camera_optical_joint_chin
- removed joint camera_optical_joint_face
- removed joint camera_optical_joint_left
- removed joint camera_optical_joint_rearDown
- removed joint camera_optical_joint_right
- removed joint ultraSound_joint_face
- removed joint ultraSound_joint_left
- removed joint ultraSound_joint_right
- joint FL_calf_joint: limit lower=-2.72271363311 upper=-0.837758040957 effort=23.7 velocity=30.1 -> lower=-2.69653369433 upper=-0.916297857297 effort=33.5 velocity=28
- joint FL_hip_joint: limit lower=-1.0471975512 upper=1.0471975512 effort=23.7 velocity=30.1 -> lower=-0.802851455917 upper=0.802851455917 effort=33.5 velocity=50
- joint FL_thigh_joint: limit lower=-0.663225115758 upper=2.96705972839 effort=23.7 velocity=30.1 -> lower=-1.0471975512 upper=4.18879020479 effort=33.5 velocity=28
- joint FR_calf_joint: limit lower=-2.72271363311 upper=-0.837758040957 effort=23.7 velocity=30.1 -> lower=-2.69653369433 upper=-0.916297857297 effort=33.5 velocity=28
- joint FR_hip_joint: limit lower=-1.0471975512 upper=1.0471975512 effort=23.7 velocity=30.1 -> lower=-0.802851455917 upper=0.802851455917 effort=33.5 velocity=50
- joint FR_thigh_joint: limit lower=-0.663225115758 upper=2.96705972839 effort=23.7 velocity=30.1 -> lower=-1.0471975512 upper=4.18879020479 effort=33.5 velocity=28
- joint RL_calf_joint: limit lower=-2.72271363311 upper=-0.837758040957 effort=23.7 velocity=30.1 -> lower=-2.69653369433 upper=-0.916297857297 effort=33.5 velocity=28
- joint RL_hip_joint: limit lower=-1.0471975512 upper=1.0471975512 effort=23.7 velocity=30.1 -> lower=-0.802851455917 upper=0.802851455917 effort=33.5 velocity=50
- joint RL_thigh_joint: limit lower=-0.663225115758 upper=2.96705972839 effort=23.7 velocity=30.1 -> lower=-1.0471975512 upper=4.18879020479 effort=33.5 velocity=28
- joint RR_calf_joint: limit lower=-2.72271363311 upper=-0.837758040957 effort=23.7 velocity=30.1 -> lower=-2.69653369433 upper=-0.916297857297 effort=33.5 velocity=28
- joint RR_hip_joint: limit lower=-1.0471975512 upper=1.0471975512 effort=23.7 velocity=30.1 -> lower=-0.802851455917 upper=0.802851455917 effort=33.5 velocity=50
- joint RR_thigh_joint: limit lower=-0.663225115758 upper=2.96705972839 effort=23.7 velocity=30.1 -> lower=-1.0471975512 upper=4.18879020479 effort=33.5 velocity=28

Commit message: add aliengo

File: resources/robots/go1/urdf/go1.urdf (robot description, URDF)
Before this commit: robot go1_description, 23 links, 22 joints
Links:
- added link camera_chin, mass 1e-5; collision box size=.001 .001 .001; visual mesh filename=../meshes/depthCamera.dae scale=1 1 1
- added link camera_face, mass 1e-5; collision box size=.001 .001 .001; visual mesh filename=../meshes/depthCamera.dae scale=1 1 1
- added link camera_laserscan_link_left
- added link camera_laserscan_link_right
- added link camera_left, mass 1e-5; collision box size=.001 .001 .001; visual mesh filename=../meshes/depthCamera.dae scale=1 1 1
- added link camera_optical_chin
- added link camera_optical_face
- added link camera_optical_left
- added link camera_optical_rearDown
- added link camera_optical_right
- added link camera_rearDown, mass 1e-5; collision box size=.001 .001 .001; visual mesh filename=../meshes/depthCamera.dae scale=1 1 1
- added link camera_right, mass 1e-5; collision box size=.001 .001 .001; visual mesh filename=../meshes/depthCamera.dae scale=1 1 1
- added link ultraSound_face, mass 1e-5; collision box size=.001 .001 .001; visual mesh filename=../meshes/ultraSound.dae scale=1 1 1
- added link ultraSound_left, mass 1e-5; collision box size=.001 .001 .001; visual mesh filename=../meshes/ultraSound.dae scale=1 1 1
- added link ultraSound_right, mass 1e-5; collision box size=.001 .001 .001; visual mesh filename=../meshes/ultraSound.dae scale=1 1 1
- link FL_calf: mass 0.158015 -> 0.131; geometry collision box size=0.213 0.016 0.016; visual mesh filename=../meshes/calf.dae scale=1 1 1
- link FL_hip: mass 0.510299 -> 0.591; geometry collision cylinder length=0.04 radius=0.046; visual mesh filename=../meshes/hip.dae scale=1 1 1
- link FL_thigh: mass 0.898919 -> 0.92; geometry collision box size=0.213 0.0245 0.034; visual mesh filename=../meshes/thigh.dae scale=1 1 1
- link FL_thigh_shoulder: geometry collision cylinder length=0.032 radius=0.041
- link FR_calf: mass 0.158015 -> 0.131; geometry collision box size=0.213 0.016 0.016; visual mesh filename=../meshes/calf.dae scale=1 1 1
- link FR_hip: mass 0.510299 -> 0.591; geometry collision cylinder length=0.04 radius=0.046; visual mesh filename=../meshes/hip.dae scale=1 1 1
- link FR_thigh: mass 0.898919 -> 0.92; geometry collision box size=0.213 0.0245 0.034; visual mesh filename=../meshes/thigh_mirror.dae scale=1 1 1
- link FR_thigh_shoulder: geometry collision cylinder length=0.032 radius=0.041
- link RL_calf: mass 0.158015 -> 0.131; geometry collision box size=0.213 0.016 0.016; visual mesh filename=../meshes/calf.dae scale=1 1 1
- link RL_hip: mass 0.510299 -> 0.591; geometry collision cylinder length=0.04 radius=0.046; visual mesh filename=../meshes/hip.dae scale=1 1 1
- link RL_thigh: mass 0.898919 -> 0.92; geometry collision box size=0.213 0.0245 0.034; visual mesh filename=../meshes/thigh.dae scale=1 1 1
- link RL_thigh_shoulder: geometry collision cylinder length=0.032 radius=0.041
- link RR_calf: mass 0.158015 -> 0.131; geometry collision box size=0.213 0.016 0.016; visual mesh filename=../meshes/calf.dae scale=1 1 1
- link RR_hip: mass 0.510299 -> 0.591; geometry collision cylinder length=0.04 radius=0.046; visual mesh filename=../meshes/hip.dae scale=1 1 1
- link RR_thigh: mass 0.898919 -> 0.92; geometry collision box size=0.213 0.0245 0.034; visual mesh filename=../meshes/thigh_mirror.dae scale=1 1 1
- link RR_thigh_shoulder: geometry collision cylinder length=0.032 radius=0.041
- link imu_link: geometry collision box size=.001 .001 .001; visual box size=0.001 0.001 0.001
- link trunk: mass 4.8 -> 5.204; geometry collision box size=0.3762 0.0935 0.114; visual mesh filename=../meshes/trunk.dae scale=1 1 1
Joints:
- added joint camera_joint_chin: type fixed, parent trunk, child camera_chin, origin xyz=0.2522 0.0125 -0.0436 rpy=3.14159265359 1.57079632679 0
- added joint camera_joint_face: type fixed, parent trunk, child camera_face, origin xyz=0.2785 0.0125 0.0167 rpy=3.14159265359 0 0
- added joint camera_joint_left: type fixed, parent trunk, child camera_left, origin xyz=-0.066 0.082 -0.0176 rpy=3.14159265359 0.2618 1.57079632679
- added joint camera_joint_rearDown: type fixed, parent trunk, child camera_rearDown, origin xyz=-0.0825 0.0125 -0.04365 rpy=3.14159265359 1.57079632679 0
- added joint camera_joint_right: type fixed, parent trunk, child camera_right, origin xyz=-0.041 -0.082 -0.0176 rpy=3.14159265359 0.2618 -1.57079632679
- added joint camera_laserscan_joint_left: type fixed, parent camera_left, child camera_laserscan_link_left, origin xyz=0 0 0 rpy=0 0.2618 0
- added joint camera_laserscan_joint_right: type fixed, parent camera_right, child camera_laserscan_link_right, origin xyz=0 0 0 rpy=0 0.2618 0
- added joint camera_optical_joint_chin: type fixed, parent camera_chin, child camera_optical_chin, origin xyz=0 0 0 rpy=-1.57079632679 0 -1.57079632679
- added joint camera_optical_joint_face: type fixed, parent camera_face, child camera_optical_face, origin xyz=0 0 0 rpy=-1.57079632679 0 -1.57079632679
- added joint camera_optical_joint_left: type fixed, parent camera_left, child camera_optical_left, origin xyz=0 0 0 rpy=-1.57079632679 0 -1.57079632679
- added joint camera_optical_joint_rearDown: type fixed, parent camera_rearDown, child camera_optical_rearDown, origin xyz=0 0 0 rpy=-1.57079632679 0 -1.57079632679
- added joint camera_optical_joint_right: type fixed, parent camera_right, child camera_optical_right, origin xyz=0 0 0 rpy=-1.57079632679 0 -1.57079632679
- added joint ultraSound_joint_face: type fixed, parent trunk, child ultraSound_face, origin xyz=0.2747 0.0 -0.0088 rpy=0 0 0
- added joint ultraSound_joint_left: type fixed, parent trunk, child ultraSound_left, origin xyz=-0.0535  0.0826 0.00868 rpy=0 0.2618 1.57079632679
- added joint ultraSound_joint_right: type fixed, parent trunk, child ultraSound_right, origin xyz=-0.0535 -0.0826 0.00868 rpy=0 0.2618 -1.57079632679
- joint FL_calf_joint: limit lower=-2.69653369433 upper=-0.916297857297 effort=33.5 velocity=28 -> lower=-2.72271363311 upper=-0.837758040957 effort=23.7 velocity=30.1
- joint FL_hip_joint: limit lower=-0.802851455917 upper=0.802851455917 effort=33.5 velocity=50 -> lower=-1.0471975512 upper=1.0471975512 effort=23.7 velocity=30.1
- joint FL_thigh_joint: limit lower=-1.0471975512 upper=4.18879020479 effort=33.5 velocity=28 -> lower=-0.663225115758 upper=2.96705972839 effort=23.7 velocity=30.1
- joint FR_calf_joint: limit lower=-2.69653369433 upper=-0.916297857297 effort=33.5 velocity=28 -> lower=-2.72271363311 upper=-0.837758040957 effort=23.7 velocity=30.1
- joint FR_hip_joint: limit lower=-0.802851455917 upper=0.802851455917 effort=33.5 velocity=50 -> lower=-1.0471975512 upper=1.0471975512 effort=23.7 velocity=30.1
- joint FR_thigh_joint: limit lower=-1.0471975512 upper=4.18879020479 effort=33.5 velocity=28 -> lower=-0.663225115758 upper=2.96705972839 effort=23.7 velocity=30.1
- joint RL_calf_joint: limit lower=-2.69653369433 upper=-0.916297857297 effort=33.5 velocity=28 -> lower=-2.72271363311 upper=-0.837758040957 effort=23.7 velocity=30.1
- joint RL_hip_joint: limit lower=-0.802851455917 upper=0.802851455917 effort=33.5 velocity=50 -> lower=-1.0471975512 upper=1.0471975512 effort=23.7 velocity=30.1
- joint RL_thigh_joint: limit lower=-1.0471975512 upper=4.18879020479 effort=33.5 velocity=28 -> lower=-0.663225115758 upper=2.96705972839 effort=23.7 velocity=30.1
- joint RR_calf_joint: limit lower=-2.69653369433 upper=-0.916297857297 effort=33.5 velocity=28 -> lower=-2.72271363311 upper=-0.837758040957 effort=23.7 velocity=30.1
- joint RR_hip_joint: limit lower=-0.802851455917 upper=0.802851455917 effort=33.5 velocity=50 -> lower=-1.0471975512 upper=1.0471975512 effort=23.7 velocity=30.1
- joint RR_thigh_joint: limit lower=-1.0471975512 upper=4.18879020479 effort=33.5 velocity=28 -> lower=-0.663225115758 upper=2.96705972839 effort=23.7 velocity=30.1

File: resources/robots/go1_description/urdf/go1.urdf (robot description, URDF)
Before this commit: robot go1_description, 38 links, 37 joints
Joints:
- joint FL_foot_fixed: type  fixed -> fixed
