Commit message: add

File: resources/robots/aliengo/urdf/aliengo.urdf (robot description, URDF)
Before this commit: robot aliengo_description, 19 links, 18 joints
Joints:
- joint FL_thigh_joint: limit lower=-1.0471975512 upper=4.18879020479 effort=44 velocity=20 -> effort=44 velocity=20; type revolute -> continuous
- joint FR_thigh_joint: limit lower=-1.0471975512 upper=4.18879020479 effort=44 velocity=20 -> effort=44 velocity=20; type revolute -> continuous
- joint RL_thigh_joint: limit lower=-1.0471975512 upper=4.18879020479 effort=44 velocity=20 -> effort=44 velocity=20; type revolute -> continuous
- joint RR_thigh_joint: limit lower=-1.0471975512 upper=4.18879020479 effort=44 velocity=20 -> effort=44 velocity=20; type revolute -> continuous
