Commit message: add new gen

File: resources/robots/go1_description/urdf/go1.urdf (robot description, URDF)
Before this commit: robot go1_description, 38 links, 37 joints
Links:
- link FL_calf: geometry collision box size=0.213 0.016 0.016; visual mesh filename=package://go1_description/meshes/calf.dae scale=1 1 1
- link FL_hip: geometry collision cylinder length=0.04 radius=0.046; visual mesh filename=package://go1_description/meshes/hip.dae scale=1 1 1
- link FL_thigh: geometry collision box size=0.213 0.0245 0.034; visual mesh filename=package://go1_description/meshes/thigh.dae scale=1 1 1
- link FR_calf: geometry collision box size=0.213 0.016 0.016; visual mesh filename=package://go1_description/meshes/calf.dae scale=1 1 1
- link FR_hip: geometry collision cylinder length=0.04 radius=0.046; visual mesh filename=package://go1_description/meshes/hip.dae scale=1 1 1
- link FR_thigh: geometry collision box size=0.213 0.0245 0.034; visual mesh filename=package://go1_description/meshes/thigh_mirror.dae scale=1 1 1
- link RL_calf: geometry collision box size=0.213 0.016 0.016; visual mesh filename=package://go1_description/meshes/calf.dae scale=1 1 1
- link RL_hip: geometry collision cylinder length=0.04 radius=0.046; visual mesh filename=package://go1_description/meshes/hip.dae scale=1 1 1
- link RL_thigh: geometry collision box size=0.213 0.0245 0.034; visual mesh filename=package://go1_description/meshes/thigh.dae scale=1 1 1
- link RR_calf: geometry collision box size=0.213 0.016 0.016; visual mesh filename=package://go1_description/meshes/calf.dae scale=1 1 1
- link RR_hip: geometry collision cylinder length=0.04 radius=0.046; visual mesh filename=package://go1_description/meshes/hip.dae scale=1 1 1
- link RR_thigh: geometry collision box size=0.213 0.0245 0.034; visual mesh filename=package://go1_description/meshes/thigh_mirror.dae scale=1 1 1
- link camera_chin: geometry collision box size=.001 .001 .001; visual mesh filename=package://go1_description/meshes/depthCamera.dae scale=1 1 1
- link camera_face: geometry collision box size=.001 .001 .001; visual mesh filename=package://go1_description/meshes/depthCamera.dae scale=1 1 1
- link camera_left: geometry collision box size=.001 .001 .001; visual mesh filename=package://go1_description/meshes/depthCamera.dae scale=1 1 1
- link camera_rearDown: geometry collision box size=.001 .001 .001; visual mesh filename=package://go1_description/meshes/depthCamera.dae scale=1 1 1
- link camera_right: geometry collision box size=.001 .001 .001; visual mesh filename=package://go1_description/meshes/depthCamera.dae scale=1 1 1
- link trunk: geometry collision box size=0.3762 0.0935 0.114; visual mesh filename=package://go1_description/meshes/trunk.dae scale=1 1 1
- link ultraSound_face: geometry collision box size=.001 .001 .001; visual mesh filename=package://go1_description/meshes/ultraSound.dae scale=1 1 1
- link ultraSound_left: geometry collision box size=.001 .001 .001; visual mesh filename=package://go1_description/meshes/ultraSound.dae scale=1 1 1
- link ultraSound_right: geometry collision box size=.001 .001 .001; visual mesh filename=package://go1_description/meshes/ultraSound.dae scale=1 1 1

Commit message: add new go1 urdf

File: resources/robots/go1_description/urdf/go1.urdf (robot description, URDF)
Before this commit: robot go1_description, 38 links, 37 joints
Links:
- link FL_calf: geometry collision box size=0.213 0.016 0.016; visual mesh filename=../meshes/calf.dae scale=1 1 1
- link FL_hip: geometry collision cylinder length=0.04 radius=0.046; visual mesh filename=../meshes/hip.dae scale=1 1 1
- link FL_thigh: geometry collision box size=0.213 0.0245 0.034; visual mesh filename=../meshes/thigh.dae scale=1 1 1
- link FR_calf: geometry collision box size=0.213 0.016 0.016; visual mesh filename=../meshes/calf.dae scale=1 1 1
- link FR_hip: geometry collision cylinder length=0.04 radius=0.046; visual mesh filename=../meshes/hip.dae scale=1 1 1
- link FR_thigh: geometry collision box size=0.213 0.0245 0.034; visual mesh filename=../meshes/thigh_mirror.dae scale=1 1 1
- link RL_calf: geometry collision box size=0.213 0.016 0.016; visual mesh filename=../meshes/calf.dae scale=1 1 1
- link RL_hip: geometry collision cylinder length=0.04 radius=0.046; visual mesh filename=../meshes/hip.dae scale=1 1 1
- link RL_thigh: geometry collision box size=0.213 0.0245 0.034; visual mesh filename=../meshes/thigh.dae scale=1 1 1
- link RR_calf: geometry collision box size=0.213 0.016 0.016; visual mesh filename=../meshes/calf.dae scale=1 1 1
- link RR_hip: geometry collision cylinder length=0.04 radius=0.046; visual mesh filename=../meshes/hip.dae scale=1 1 1
- link RR_thigh: geometry collision box size=0.213 0.0245 0.034; visual mesh filename=../meshes/thigh_mirror.dae scale=1 1 1
- link camera_chin: geometry collision box size=.001 .001 .001; visual mesh filename=../meshes/depthCamera.dae scale=1 1 1
- link camera_face: geometry collision box size=.001 .001 .001; visual mesh filename=../meshes/depthCamera.dae scale=1 1 1
- link camera_left: geometry collision box size=.001 .001 .001; visual mesh filename=../meshes/depthCamera.dae scale=1 1 1
- link camera_rearDown: geometry collision box size=.001 .001 .001; visual mesh filename=../meshes/depthCamera.dae scale=1 1 1
- link camera_right: geometry collision box size=.001 .001 .001; visual mesh filename=../meshes/depthCamera.dae scale=1 1 1
- link trunk: geometry collision box size=0.3762 0.0935 0.114; visual mesh filename=../meshes/trunk.dae scale=1 1 1
- link ultraSound_face: geometry collision box size=.001 .001 .001; visual mesh filename=../meshes/ultraSound.dae scale=1 1 1
- link ultraSound_left: geometry collision box size=.001 .001 .001; visual mesh filename=../meshes/ultraSound.dae scale=1 1 1
- link ultraSound_right: geometry collision box size=.001 .001 .001; visual mesh filename=../meshes/ultraSound.dae scale=1 1 1

File: resources/robots/go2/urdf/go1.urdf (robot description, URDF)
Before this commit: robot go1_description, 23 links, 22 joints
Links:
- link FL_calf: geometry collision box size=0.213 0.016 0.016; visual mesh filename=../meshes/calf.dae scale=1 1 1
- link FL_hip: geometry collision cylinder length=0.04 radius=0.046; visual mesh filename=../meshes/hip.dae scale=1 1 1
- link FL_thigh: geometry collision box size=0.213 0.0245 0.034; visual mesh filename=../meshes/thigh.dae scale=1 1 1
- link FR_calf: geometry collision box size=0.213 0.016 0.016; visual mesh filename=../meshes/calf.dae scale=1 1 1
- link FR_hip: geometry collision cylinder length=0.04 radius=0.046; visual mesh filename=../meshes/hip.dae scale=1 1 1
- link FR_thigh: geometry collision box size=0.213 0.0245 0.034; visual mesh filename=../meshes/thigh_mirror.dae scale=1 1 1
- link RL_calf: geometry collision box size=0.213 0.016 0.016; visual mesh filename=../meshes/calf.dae scale=1 1 1
- link RL_hip: geometry collision cylinder length=0.04 radius=0.046; visual mesh filename=../meshes/hip.dae scale=1 1 1
- link RL_thigh: geometry collision box size=0.213 0.0245 0.034; visual mesh filename=../meshes/thigh.dae scale=1 1 1
- link RR_calf: geometry collision box size=0.213 0.016 0.016; visual mesh filename=../meshes/calf.dae scale=1 1 1
- link RR_hip: geometry collision cylinder length=0.04 radius=0.046; visual mesh filename=../meshes/hip.dae scale=1 1 1
- link RR_thigh: geometry collision box size=0.213 0.0245 0.034; visual mesh filename=../meshes/thigh_mirror.dae scale=1 1 1
- link trunk: geometry collision box size=0.3762 0.0935 0.114; visual mesh filename=../meshes/trunk.dae scale=1 1 1
