Commit message: ablation_study

File: resources/robots/aliengo_description/urdf/aliengo.urdf (robot description, URDF)
Before this commit: robot aliengo_description, 19 links, 18 joints
Links:
- added link FL_calf_rotor, mass 0.132; collision cylinder length=0.02 radius=0.035; visual cylinder length=0.02 radius=0.035
- added link FL_hip_rotor, mass 0.146; collision cylinder length=0.02 radius=0.035; visual cylinder length=0.02 radius=0.035
- added link FL_thigh_rotor, mass 0.146; collision cylinder length=0.02 radius=0.035; visual cylinder length=0.02 radius=0.035
- added link FR_calf_rotor, mass 0.132; collision cylinder length=0.02 radius=0.035; visual cylinder length=0.02 radius=0.035
- added link FR_hip_rotor, mass 0.146; collision cylinder length=0.02 radius=0.035; visual cylinder length=0.02 radius=0.035
- added link FR_thigh_rotor, mass 0.146; collision cylinder length=0.02 radius=0.035; visual cylinder length=0.02 radius=0.035
- added link RL_calf_rotor, mass 0.132; collision cylinder length=0.02 radius=0.035; visual cylinder length=0.02 radius=0.035
- added link RL_hip_rotor, mass 0.146; collision cylinder length=0.02 radius=0.035; visual cylinder length=0.02 radius=0.035
- added link RL_thigh_rotor, mass 0.146; collision cylinder length=0.02 radius=0.035; visual cylinder length=0.02 radius=0.035
- added link RR_calf_rotor, mass 0.132; collision cylinder length=0.02 radius=0.035; visual cylinder length=0.02 radius=0.035
- added link RR_hip_rotor, mass 0.146; collision cylinder length=0.02 radius=0.035; visual cylinder length=0.02 radius=0.035
- added link RR_thigh_rotor, mass 0.146; collision cylinder length=0.02 radius=0.035; visual cylinder length=0.02 radius=0.035
- link trunk: mass 9.041 -> 11.644
Joints:
- added joint FL_calf_rotor_joint: type fixed, parent FL_thigh, child FL_calf_rotor, origin xyz=0.0 -0.0997 0 rpy=0 0 0
- added joint FL_hip_rotor_joint: type fixed, parent trunk, child FL_hip_rotor, origin xyz=0.139985 0.051 0 rpy=0 0 0
- added joint FL_thigh_rotor_joint: type fixed, parent FL_hip, child FL_thigh_rotor, origin xyz=0.0 0.0298 0 rpy=0 0 0
- added joint FR_calf_rotor_joint: type fixed, parent FR_thigh, child FR_calf_rotor, origin xyz=0.0 0.0997 0 rpy=0 0 0
- added joint FR_hip_rotor_joint: type fixed, parent trunk, child FR_hip_rotor, origin xyz=0.139985 -0.051 0 rpy=0 0 0
- added joint FR_thigh_rotor_joint: type fixed, parent FR_hip, child FR_thigh_rotor, origin xyz=0.0 -0.0298 0 rpy=0 0 0
- added joint RL_calf_rotor_joint: type fixed, parent RL_thigh, child RL_calf_rotor, origin xyz=0.0 -0.0997 0 rpy=0 0 0
- added joint RL_hip_rotor_joint: type fixed, parent trunk, child RL_hip_rotor, origin xyz=-0.139985 0.051 0 rpy=0 0 0
- added joint RL_thigh_rotor_joint: type fixed, parent RL_hip, child RL_thigh_rotor, origin xyz=0.0 0.0298 0 rpy=0 0 0
- added joint RR_calf_rotor_joint: type fixed, parent RR_thigh, child RR_calf_rotor, origin xyz=0.0 0.0997 0 rpy=0 0 0
- added joint RR_hip_rotor_joint: type fixed, parent trunk, child RR_hip_rotor, origin xyz=-0.139985 -0.051 0 rpy=0 0 0
- added joint RR_thigh_rotor_joint: type fixed, parent RR_hip, child RR_thigh_rotor, origin xyz=0.0 -0.0298 0 rpy=0 0 0
- joint FL_calf_joint: limit lower=-2.77507351067 upper=-0.645771823238 effort=55 velocity=16 -> lower=-2.775073510670984 upper=-0.6457718232379019 effort=44.4 velocity=15.89
- joint FL_hip_joint: limit lower=-1.2217304764 upper=1.2217304764 effort=44 velocity=20 -> lower=-1.2217304763960306 upper=1.2217304763960306 effort=35.278 velocity=20; origin xyz=0.2399 0.051 0 rpy=0 0 0 -> xyz=0.2407 0.051 0 rpy=0 0 0
- joint FL_thigh_joint: limit lower=-1.0471975512 upper=4.18879020479 effort=44 velocity=20 -> effort=35.278 velocity=20; origin xyz=0 0.083 0 rpy=0 0 0 -> xyz=0 0.0868 0 rpy=0 0 0; type revolute -> continuous
- joint FR_calf_joint: limit lower=-2.77507351067 upper=-0.645771823238 effort=55 velocity=16 -> lower=-2.775073510670984 upper=-0.6457718232379019 effort=44.4 velocity=15.89
- joint FR_hip_joint: limit lower=-1.2217304764 upper=1.2217304764 effort=44 velocity=20 -> lower=-1.2217304763960306 upper=1.2217304763960306 effort=35.278 velocity=20; origin xyz=0.2399 -0.051 0 rpy=0 0 0 -> xyz=0.2407 -0.051 0 rpy=0 0 0
- joint FR_thigh_joint: limit lower=-1.0471975512 upper=4.18879020479 effort=44 velocity=20 -> effort=35.278 velocity=20; origin xyz=0 -0.083 0 rpy=0 0 0 -> xyz=0 -0.0868 0 rpy=0 0 0; type revolute -> continuous
- joint RL_calf_joint: limit lower=-2.77507351067 upper=-0.645771823238 effort=55 velocity=16 -> lower=-2.775073510670984 upper=-0.6457718232379019 effort=44.4 velocity=15.89
- joint RL_hip_joint: limit lower=-1.2217304764 upper=1.2217304764 effort=44 velocity=20 -> lower=-1.2217304763960306 upper=1.2217304763960306 effort=35.278 velocity=20; origin xyz=-0.2399 0.051 0 rpy=0 0 0 -> xyz=-0.2407 0.051 0 rpy=0 0 0
- joint RL_thigh_joint: limit lower=-1.0471975512 upper=4.18879020479 effort=44 velocity=20 -> effort=35.278 velocity=20; origin xyz=0 0.083 0 rpy=0 0 0 -> xyz=0 0.0868 0 rpy=0 0 0; type revolute -> continuous
- joint RR_calf_joint: limit lower=-2.77507351067 upper=-0.645771823238 effort=55 velocity=16 -> lower=-2.775073510670984 upper=-0.6457718232379019 effort=44.4 velocity=15.89
- joint RR_hip_joint: limit lower=-1.2217304764 upper=1.2217304764 effort=44 velocity=20 -> lower=-1.2217304763960306 upper=1.2217304763960306 effort=35.278 velocity=20; origin xyz=-0.2399 -0.051 0 rpy=0 0 0 -> xyz=-0.2407 -0.051 0 rpy=0 0 0
- joint RR_thigh_joint: limit lower=-1.0471975512 upper=4.18879020479 effort=44 velocity=20 -> effort=35.278 velocity=20; origin xyz=0 -0.083 0 rpy=0 0 0 -> xyz=0 -0.0868 0 rpy=0 0 0; type revolute -> continuous
